File: hardware/ring-flex-v1/kicad/ring-flex-v1.kicad_pcb (KiCad board)
At the start: 2 copper layers, 65 x 10 mm, 0 parts

Commit message: Hardware: board regenerated from a script, islands rebudgeted
The board is now produced by kicad/gen_pcb.py rather than being a one-off
file, so the outline and zones can be regenerated as the design moves.

The island budget changed because of how the antenna keep-out works. Put the
module flush against x=0 with its antenna facing the board edge and the
datasheet's 12.4 x 3.8 mm "no ground pad" area falls off the board -- there
is no host copper there because there is no board there. The 3.8 mm I had
written off as lost is free, which is what lets the power section have a
proper island:

  [A: module 15.5] -3.5- [B: power 12] -3.5- [C: cell 16] -3.5- [D: motor 11]

54.5 mm of parts and 10.5 mm of bends: 65.0 mm exactly.

The first 3.8 mm is still marked no-copper on User.1, since the module
overhangs it. The board also now carries the flex rules, the stiffener note
and the bend-zone prohibition as text, so they are in front of whoever lays
it out.

Footprints are deliberately not placed by the script. F8 brings them in with
their nets; positioning them is a judgement call about bend zones, part
orientation and strain relief, and a generated placement would pass DRC
while failing in the fold.

DRC: 0 violations.

Co-Authored-By: Claude Opus 5 <noreply@anthropic.com>
Other:
- board text added: "A: MODULE U1 (antenna at x=0, flush to the edge)"
- board text added: "ANTENNA (User.1): no copper either layer. Datasheet keep-out is 12.4 x 3.8 mm; the board ends there."
- board text added: "B: POWER U2 U3 U4 Q1 R3 R4 R5 C2..C6"
- board text added: "BEND ZONES: no vias, no pads, no component edges. Hatched pour only, traces perpendicular and curved."
- board text added: "C: CELL BT1 16 x 8 mm"
- board text added: "D: MOTOR M1 + Q2 R1 R2 D1 C1, charge pads J1 J2"
- board text added: "Press F8 to bring footprints in from the schematic, then place them on the islands."
- board text added: "STIFFENERS under islands A, B, C and D. Static bend radius >= 6x stack thickness."
- board text added: "bend"
- board text added: "ring-flex-v1 65.0 x 10.0 mm 2-layer polyimide closed ring, index finger, 65 mm"
- board text removed: "ANTENNA KEEP-OUT: no copper, no cell, no motor"
- board text removed: "BEND"
- board text removed: "BEND ZONES: no vias, no pads, no component edges. Hatched pour only."
- board text removed: "ISLAND A: module + power (stiffener)"
- board text removed: "ISLAND B: cell (stiffener)"
- board text removed: "ISLAND C: motor (stiffener)"
- board text removed: "charge contacts"
- board text removed: "ring-flex-v1 65.0 x 10.0 mm 2-layer polyimide closed ring, index finger"
Changed lines of the file:
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@@
 		(layer "Dwgs.User")
 	)
-	(gr_text "ISLAND A: module + power  (stiffener)"
-		(at 50.500 72.000 0)
-		(layer "Cmts.User")
-		(effects
-			(font
-				(size 0.80 0.80)
-				(thickness 0.15)
-			)
-			(justify left)
-		)
-	)
-	(gr_line
-		(start 72.000 60.000)
-		(end 72.000 70.000)
-		(stroke
-			(width 0.080)
-			(type solid)
-		)
-		(layer "Dwgs.User")
-	)
-	(gr_text "BEND"
-		(at 72.500 72.000 0)
-		(layer "Cmts.User")
-		(effects
-			(font
-				(size 0.80 0.80)
-				(thickness 0.15)
-			)
-			(justify left)
-		)
-	)
-	(gr_line
-		(start 76.000 60.000)
-		(end 76.000 70.000)
-		(stroke
-			(width 0.080)
-			(type solid)
-		)
-		(layer "Dwgs.User")
-	)
-	(gr_text "ISLAND B: cell  (stiffener)"
-		(at 76.500 72.000 0)
-		(layer "Cmts.User")
-		(effects
-			(font
-				(size 0.80 0.80)
-				(thickness 0.15)
-			)
-			(justify left)
-		)
-	)
-	(gr_line
-		(start 92.000 60.000)
-		(end 92.000 70.000)
-		(stroke
-			(width 0.080)
-			(type solid)
-		)
-		(layer "Dwgs.User")
-	)
-	(gr_text "BEND"
-		(at 92.500 72.000 0)
-		(layer "Cmts.User")
-		(effects
-			(font
-				(size 0.80 0.80)
-				(thickness 0.15)
-			)
-			(justify left)
-		)
-	)
-	(gr_line
-		(start 96.000 60.000)
-		(end 96.000 70.000)
-		(stroke
-			(width 0.080)
-			(type solid)
-		)
-		(layer "Dwgs.User")
-	)
-	(gr_text "ISLAND C: motor  (stiffener)"
-		(at 96.500 72.000 0)
-		(layer "Cmts.User")
-		(effects
-			(font
-				(size 0.80 0.80)
-				(thickness 0.15)
-			)
-			(justify left)
-		)
-	)
-	(gr_line
-		(start 107.000 60.000)
-		(end 107.000 70.000)
-		(stroke
-			(width 0.080)
-			(type solid)
-		)
-		(layer "Dwgs.User")
-	)
-	(gr_text "BEND"
-		(at 107.500 72.000 0)
-		(layer "Cmts.User")
-		(effects
-			(font
-				(size 0.80 0.80)
-				(thickness 0.15)
-			)
-			(justify left)
-		)
-	)
-	(gr_line
-		(start 111.000 60.000)
-		(end 111.000 70.000)
-		(stroke
-			(width 0.080)
-			(type solid)
-		)
-		(layer "Dwgs.User")
-	)
-	(gr_text "charge contacts"
-		(at 111.500 72.000 0)
-		(layer "Cmts.User")
-		(effects
-			(font
-				(size 0.80 0.80)
+	(gr_text "A: MODULE U1  (antenna at x=0, flush to the edge)"
+		(at 50.400 72.200 0)
+		(layer "Cmts.User")
+		(effects
+			(font
+				(size 0.70 0.70)
+				(thickness 0.15)
+			)
+			(justify left)
+		)
+	)
+	(gr_line
+		(start 65.500 60.000)
+		(end 65.500 70.000)
+		(stroke
+			(width 0.080)
+			(type solid)
+		)
+		(layer "Dwgs.User")
+	)
+	(gr_text "bend"
+		(at 65.900 72.200 0)
+		(layer "Cmts.User")
+		(effects
+			(font
+				(size 0.70 0.70)
+				(thickness 0.15)
+			)
+			(justify left)
+		)
+	)
+	(gr_line
+		(start 69.000 60.000)
+		(end 69.000 70.000)
+		(stroke
+			(width 0.080)
+			(type solid)
+		)
+		(layer "Dwgs.User")
+	)
+	(gr_text "B: POWER  U2 U3 U4 Q1 R3 R4 R5 C2..C6"
+		(at 69.400 72.200 0)
+		(layer "Cmts.User")
+		(effects
+			(font
+				(size 0.70 0.70)
+				(thickness 0.15)
+			)
+			(justify left)
+		)
+	)
+	(gr_line
+		(start 81.000 60.000)
+		(end 81.000 70.000)
+		(stroke
+			(width 0.080)
+			(type solid)
+		)
+		(layer "Dwgs.User")
+	)
+	(gr_text "bend"
+		(at 81.400 72.200 0)
+		(layer "Cmts.User")
+		(effects
+			(font
+				(size 0.70 0.70)
+				(thickness 0.15)
+			)
+			(justify left)
+		)
+	)
+	(gr_line
+		(start 84.500 60.000)
+		(end 84.500 70.000)
+		(stroke
+			(width 0.080)
+			(type solid)
+		)
+		(layer "Dwgs.User")
+	)
+	(gr_text "C: CELL BT1  16 x 8 mm"
+		(at 84.900 72.200 0)
+		(layer "Cmts.User")
+		(effects
+			(font
+				(size 0.70 0.70)
+				(thickness 0.15)
+			)
+			(justify left)
+		)
+	)
+	(gr_line
+		(start 100.500 60.000)
+		(end 100.500 70.000)
+		(stroke
+			(width 0.080)
+			(type solid)
+		)
+		(layer "Dwgs.User")
+	)
+	(gr_text "bend"
+		(at 100.900 72.200 0)
+		(layer "Cmts.User")
+		(effects
+			(font
+				(size 0.70 0.70)
+				(thickness 0.15)
+			)
+			(justify left)
+		)
+	)
+	(gr_line
+		(start 104.000 60.000)
+		(end 104.000 70.000)
+		(stroke
+			(width 0.080)
+			(type solid)
+		)
+		(layer "Dwgs.User")
+	)
+	(gr_text "D: MOTOR M1 + Q2 R1 R2 D1 C1, charge pads J1 J2"
+		(at 104.400 72.200 0)
+		(layer "Cmts.User")
+		(effects
+			(font
+				(size 0.70 0.70)
 				(thickness 0.15)
 			)
@@
 	(gr_line
 		(start 50.000 60.000)
-		(end 60.000 60.000)
+		(end 53.800 60.000)
 		(stroke
 			(width 0.150)
@@
 	)
 	(gr_line
-		(start 60.000 60.000)
-		(end 60.000 70.000)
+		(start 53.800 60.000)
+		(end 53.800 70.000)
 		(stroke
 			(width 0.150)
@@
 	)
 	(gr_line
-		(start 60.000 70.000)
+		(start 53.800 70.000)
 		(end 50.000 70.000)
 		(stroke
@@
 		(layer "User.1")
 	)
-	(gr_text "ANTENNA KEEP-OUT: no copper, no cell, no motor"
-		(at 50.500 75.000 0)
-		(layer "Cmts.User")
-		(effects
-			(font
-				(size 0.90 0.90)
-				(thickness 0.15)
-			)
-			(justify left)
-		)
-	)
-	(gr_text "ring-flex-v1  65.0 x 10.0 mm  2-layer polyimide  closed ring, index finger"
+	(gr_text "ring-flex-v1   65.0 x 10.0 mm   2-layer polyimide   closed ring, index finger, 65 mm"
+		(at 50.000 52.000 0)
+		(layer "Cmts.User")
+		(effects
+			(font
+				(size 0.90 0.90)
+				(thickness 0.15)
+			)
+			(justify left)
+		)
+	)
+	(gr_text "BEND ZONES: no vias, no pads, no component edges. Hatched pour only, traces perpendicular and curved."
+		(at 50.000 54.000 0)
+		(layer "Cmts.User")
+		(effects
+			(font
+				(size 0.90 0.90)
+				(thickness 0.15)
+			)
+			(justify left)
+		)
+	)
+	(gr_text "ANTENNA (User.1): no copper either layer. Datasheet keep-out is 12.4 x 3.8 mm; the board ends there."
 		(at 50.000 56.000 0)
 		(layer "Cmts.User")
 		(effects
 			(font
-				(size 1.10 1.10)
-				(thickness 0.15)
-			)
-			(justify left)
-		)
-	)
-	(gr_text "BEND ZONES: no vias, no pads, no component edges. Hatched pour only."
+				(size 0.90 0.90)
+				(thickness 0.15)
+			)
+			(justify left)
+		)
+	)
+	(gr_text "STIFFENERS under islands A, B, C and D. Static bend radius >= 6x stack thickness."
 		(at 50.000 58.000 0)
 		(layer "Cmts.User")
 		(effects
+			(font
+				(size 0.90 0.90)
+				(thickness 0.15)
+			)
+			(justify left)
+		)
+	)
+	(gr_text "Press F8 to bring footprints in from the schematic, then place them on the islands."
+		(at 50.000 60.000 0)
+		(layer "Cmts.User")
+		(effects
